File: PCB/BSPD-07/BSPD-07.kicad_sch (KiCad schematic)
At the start: 54 parts, among them IC1 LM393LVQDRQ1, IC2 LM393LVQDRQ1, IC3 LM393LVQDRQ1, IC4 LDO40LPU50RY, IC5 74LVC1G02GW-Q100H, J1 DTM13-12PA, Q1 RSQ025P03HZGTR, Q2 RJU002N06FRAT106, Q3 RJU002N06FRAT106, U2 TLP175A / COMUS AB38-Q

Commit message: 500ms section layout
Connections:
- net 500MS_REF: now reaches IC3.3 (IN1+), R11.1, R13.1
Other:
- moved on the sheet: R11, R13
Changed lines of the file:
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@@
   (junction (at 256.54 52.07) (diameter 0) (color 0 0 0 0)
   )
-  (junction (at 179.705 38.735) (diameter 0) (color 0 0 0 0)
+  (junction (at 175.895 38.735) (diameter 0) (color 0 0 0 0)
   )
   (junction (at 179.705 41.275) (diameter 0) (color 0 0 0 0)
@@
     (stroke (width 0) (type default) (color 0 0 0 0))
   )
-  (wire (pts (xy 177.8 38.735) (xy 179.705 38.735))
+  (wire (pts (xy 173.99 38.735) (xy 175.895 38.735))
     (stroke (width 0) (type default) (color 0 0 0 0))
   )
@@
     (stroke (width 0) (type default) (color 0 0 0 0))
   )
-  (wire (pts (xy 179.705 31.115) (xy 179.705 32.385))
+  (wire (pts (xy 175.895 31.115) (xy 175.895 32.385))
     (stroke (width 0) (type default) (color 0 0 0 0))
   )
@@
     (stroke (width 0) (type default) (color 0 0 0 0))
   )
+  (wire (pts (xy 175.895 38.735) (xy 182.245 38.735))
+    (stroke (width 0) (type default) (color 0 0 0 0))
+  )
   (wire (pts (xy 210.185 42.545) (xy 212.725 42.545))
     (stroke (width 0) (type default) (color 0 0 0 0))
@@
     (stroke (width 0) (type default) (color 0 0 0 0))
   )
-  (wire (pts (xy 179.705 37.465) (xy 179.705 38.735))
+  (wire (pts (xy 175.895 37.465) (xy 175.895 38.735))
     (stroke (width 0) (type default) (color 0 0 0 0))
   )
@@
     (stroke (width 0) (type default) (color 0 0 0 0))
   )
-  (wire (pts (xy 179.705 38.735) (xy 182.245 38.735))
-    (stroke (width 0) (type default) (color 0 0 0 0))
-  )
   (wire (pts (xy 184.785 64.135) (xy 186.69 64.135))
     (stroke (width 0) (type default) (color 0 0 0 0))
@@
     (stroke (width 0) (type default) (color 0 0 0 0))
   )
-  (wire (pts (xy 170.815 38.735) (xy 172.72 38.735))
+  (wire (pts (xy 167.005 38.735) (xy 168.91 38.735))
     (stroke (width 0) (type default) (color 0 0 0 0))
   )
@@
   (text "BSPD for PGR-07 (2023)" (at 186.69 191.135 0)
     (effects (font (size 1.6 1.6) (thickness 0.32) bold italic) (justify left bottom))
+  )
+  (label "500MS_REF" (at 177.165 38.735 0)
+    (effects (font (size 0.6 0.6)) (justify left bottom))
   )
   (global_label "TPS_IN" (shape input) (at 34.925 40.64 180) (fields_autoplaced)
@@
     )
   )
-  (symbol (lib_id "power:+5V") (at 179.705 31.115 0) (unit 1)
-    (in_bom yes) (on_board yes) (fields_autoplaced)
-    (property "Reference" "#PWR0125" (id 0) (at 179.705 34.925 0)
-      (effects (font (size 1.27 1.27)) hide)
-    )
-    (property "Value" "+5V" (id 1) (at 179.705 26.67 0))
-    (property "Footprint" "" (id 2) (at 179.705 31.115 0)
-      (effects (font (size 1.27 1.27)) hide)
-    )
-    (property "Datasheet" "" (id 3) (at 179.705 31.115 0)
+  (symbol (lib_id "power:+5V") (at 175.895 31.115 0) (unit 1)
+    (in_bom yes) (on_board yes) (fields_autoplaced)
+    (property "Reference" "#PWR0125" (id 0) (at 175.895 34.925 0)
+      (effects (font (size 1.27 1.27)) hide)
+    )
+    (property "Value" "+5V" (id 1) (at 175.895 26.67 0))
+    (property "Footprint" "" (id 2) (at 175.895 31.115 0)
+      (effects (font (size 1.27 1.27)) hide)
+    )
+    (property "Datasheet" "" (id 3) (at 175.895 31.115 0)
       (effects (font (size 1.27 1.27)) hide)
     )
@@
     (pin "1")
   )
-  (symbol (lib_id "Device:R_Small") (at 175.26 38.735 270) (unit 1)
-    (in_bom yes) (on_board yes)
-    (property "Reference" "R11" (id 0) (at 175.26 34.925 90))
-    (property "Value" "100k" (id 1) (at 175.26 36.83 90))
-    (property "Footprint" "Resistor_SMD:R_0402_1005Metric" (id 2) (at 175.26 38.735 0)
-      (effects (font (size 1.27 1.27)) hide)
-    )
-    (property "Datasheet" "~" (id 3) (at 175.26 38.735 0)
+  (symbol (lib_id "Device:R_Small") (at 171.45 38.735 270) (unit 1)
+    (in_bom yes) (on_board yes)
+    (property "Reference" "R11" (id 0) (at 171.45 34.925 90))
+    (property "Value" "100k" (id 1) (at 171.45 36.83 90))
+    (property "Footprint" "Resistor_SMD:R_0402_1005Metric" (id 2) (at 171.45 38.735 0)
+      (effects (font (size 1.27 1.27)) hide)
+    )
+    (property "Datasheet" "~" (id 3) (at 171.45 38.735 0)
       (effects (font (size 1.27 1.27)) hide)
     )
@@
     (pin "2")
   )
-  (symbol (lib_id "Device:R_Small") (at 179.705 34.925 180) (unit 1)
-    (in_bom yes) (on_board yes)
-    (property "Reference" "R13" (id 0) (at 180.975 33.655 0)
+  (symbol (lib_id "Device:R_Small") (at 175.895 34.925 180) (unit 1)
+    (in_bom yes) (on_board yes)
+    (property "Reference" "R13" (id 0) (at 177.165 33.655 0)
       (effects (font (size 1.27 1.27)) (justify right))
     )
-    (property "Value" "39k" (id 1) (at 180.975 35.56 0)
+    (property "Value" "39k" (id 1) (at 177.165 35.56 0)
       (effects (font (size 1.27 1.27)) (justify right))
     )
-    (property "Footprint" "Resistor_SMD:R_0402_1005Metric" (id 2) (at 179.705 34.925 0)
-      (effects (font (size 1.27 1.27)) hide)
-    )
-    (property "Datasheet" "~" (id 3) (at 179.705 34.925 0)
+    (property "Footprint" "Resistor_SMD:R_0402_1005Metric" (id 2) (at 175.895 34.925 0)
+      (effects (font (size 1.27 1.27)) hide)
+    )
+    (property "Datasheet" "~" (id 3) (at 175.895 34.925 0)
       (effects (font (size 1.27 1.27)) hide)
     )
@@
     (pin "1")
   )
-  (symbol (lib_id "power:GND") (at 170.815 38.735 270) (unit 1)
-    (in_bom yes) (on_board yes) (fields_autoplaced)
-    (property "Reference" "#PWR0124" (id 0) (at 164.465 38.735 0)
-      (effects (font (size 1.27 1.27)) hide)
-    )
-    (property "Value" "GND" (id 1) (at 167.005 38.7349 90)
+  (symbol (lib_id "power:GND") (at 167.005 38.735 270) (unit 1)
+    (in_bom yes) (on_board yes) (fields_autoplaced)
+    (property "Reference" "#PWR0124" (id 0) (at 160.655 38.735 0)
+      (effects (font (size 1.27 1.27)) hide)
+    )
+    (property "Value" "GND" (id 1) (at 163.195 38.7349 90)
       (effects (font (size 1.27 1.27)) (justify right))
     )
-    (property "Footprint" "" (id 2) (at 170.815 38.735 0)
-      (effects (font (size 1.27 1.27)) hide)
-    )
-    (property "Datasheet" "" (id 3) (at 170.815 38.735 0)
-      (effects (font (size 1.27 1.27)) hide)
-    )
+    (property "Footprint" "" (id 2) (at 167.005 38.735 0)
+      (effects (font (size 1.27 1.27)) hide)
+    )
+    (property "Datasheet" "" (id 3) (at 167.005 38.735 0)
+      (effects (font (size 1.27 1.27)) hide)
+    )
