File: PCB/BSPD-07/BSPD-07.kicad_pcb (KiCad board)
At the start: 2 copper layers, 32 x 70.6 mm, 54 parts, among them IC1 LM393LVQDRQ1, IC2 LM393LVQDRQ1, IC3 LM393LVQDRQ1, IC4 LDO40LPU50RY, IC5 74LVC1G02GW-Q100H, J1 DTM13-12PA, Q1 RSQ025P03HZGTR, Q2 RJU002N06FRAT106, Q3 RJU002N06FRAT106, U2 TLP175A / COMUS AB38-Q

Commit message: 500ms section layout
Parts:
- moved Q1 65.3 mm to (156.8, 129.6), turned to -90 degrees
- moved R16 55.4 mm to (153.6, 127.5)
- moved IC4 52.7 mm to (158.8, 102.4), turned to 90 degrees
- moved R12 2.78 mm to (158.1, 124.4), turned to 90 degrees
- moved C3 1.67 mm to (156.3, 125.2), turned to 90 degrees
- moved R11 1.12 mm to (153.3, 124.4), turned to 90 degrees
- moved R13 0.87 mm to (154.5, 124.4), turned to 90 degrees
- moved IC3 0.62 mm to (148.7, 125.7)
- moved TP4 0.52 mm to (157.2, 121.7)
Connections:
- net Net-(IC3-Pad3) renamed /500MS_REF
Routing:
- net Net-(C3-Pad1): track 0.00 -> 7.87 mm
- net ERR_CURRENT: track 0.00 -> 5.05 mm
- net GND: track 15.1 -> 18.9 mm, vias 9 -> 12
- net /500MS_REF: track 0.00 -> 3.18 mm
- net Net-(IC3-Pad1): track 0.00 -> 1.76 mm

Commit message: Almost finished schematics
Parts:
- moved LED1 72.5 mm to (144.5, 134.0)
- moved U2 68.0 mm to (141.2, 128.2), turned to 90 degrees
- moved R14 66.4 mm to (162.0, 130.3), turned to 180 degrees
- moved R17 65.6 mm to (162.0, 127.3)
- moved C5 63.8 mm to (157.7, 128.5), turned to 180 degrees
- moved R15 62.2 mm to (162.0, 131.7)
- moved Q2 61.8 mm to (155.0, 131.4)
- moved R18 61.6 mm to (148.9, 126.5), turned to -90 degrees
- moved R21 58.6 mm to (154.3, 133.6), turned to 180 degrees
- moved Q3 55.4 mm to (148.9, 130.2), turned to -90 degrees
- moved C7 53.4 mm to (147.1, 102.3), turned to 90 degrees
- moved RV1 52.1 mm to (143.2, 118.9), turned to 90 degrees
- moved RV2 52.1 mm to (143.1, 110.8), turned to 90 degrees
- moved R26 51.3 mm to (151.9, 121.6), turned to 90 degrees
- moved R20 50.5 mm to (154.3, 129.3), turned to 180 degrees
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Connections:
- net Net-(C5-Pad2) renamed /10ms VAL
- net Net-(IC3-Pad5) renamed /10s REF
- R17 pad 1: Net-(Q1-Pad3) -> Net-(IC3-Pad1)
Routing:
- net /10ms VAL: track 0.00 -> 17.3 mm
- net Net-(Q1-Pad1): track 0.00 -> 7.89 mm
- net GND: track 18.9 -> 23.2 mm, vias 12 -> 17
- net Net-(IC3-Pad7): track 0.00 -> 4.27 mm
- net /10s REF: track 0.00 -> 3.65 mm
- net Net-(C8-Pad2): track 0.00 -> 3.11 mm
- net Net-(Q1-Pad3): track 0.00 -> 1.92 mm
- net Net-(Q2-Pad2): track 0.00 -> 1.67 mm
- net Net-(IC3-Pad1): track 1.76 -> 3.08 mm
- net +5V: track 7.04 -> 5.95 mm
Other:
- board size 32 x 70.6 mm -> 32 x 70.9 mm
